Commit message: Fixed degree_to_radian conversion issue

File: urdf/_t265.urdf.xacro (robot description, xacro)
@@ -16,4 +16,5 @@
     <xacro:property name="fisheye1_offset_y" value="0.0"/>
     <xacro:property name="fisheye1_offset_z" value="0.0"/>
+    <xacro:property name="deg_to_rad" value="0.0174533"/>
     <xacro:property name="fisheye2_offset_x" value="0.0229"/>
     <xacro:property name="fisheye2_offset_y" value="0.0"/>
