Commit message: Added D435 IMU state transform publisher.
ToDo: Publish IMU message.

File: urdf/_d435.gazebo.xacro (robot description, xacro)
@@ -6,5 +6,5 @@
 -->
 <robot xmlns:xacro="http://ros.org/wiki/xacro">
-  <xacro:macro name="gazebo_d435" params="camera_name reference_link topics_ns depth_optical_frame color_optical_frame infrared1_optical_frame infrared2_optical_frame publish_pointcloud:=true" >
+  <xacro:macro name="gazebo_d435" params="camera_name reference_link topics_ns depth_optical_frame color_optical_frame infrared1_optical_frame infrared2_optical_frame imu_optical_frame publish_pointcloud:=true" >
     <!-- Load parameters to model's main link-->
     <xacro:property name="deg_to_rad" value="0.01745329251994329577" />
@@ -137,4 +137,22 @@
       </plugin>
     </gazebo>
+    <!-- Todo: Imu data is not published -->
+    <gazebo>
+      <sensor name="${camera_name}imu" type="imu">
+        <always_on>true</always_on>
+        <update_rate>100</update_rate>
+        <topic>__default_topic__</topic>
+        <plugin name="${topics_ns}" filename="libgazebo_ros_imu_sensor.so">
+          <initial_orientation_as_reference>false</initial_orientation_as_reference>
+          <topicName>${imu_optical_frame}</topicName>
+          <bodyName>${imu_optical_frame}</bodyName>
+          <updateRateHZ>100.0</updateRateHZ>
+          <gaussianNoise>0.0</gaussianNoise>
+          <xyzOffset>0 0 0</xyzOffset>
+          <rpyOffset>0 0 0</rpyOffset>
+          <frameName>${imu_optical_frame}</frameName>
+        </plugin>
+      </sensor>
+    </gazebo>
   </xacro:macro>
 </robot>

File: urdf/_d435.urdf.xacro (robot description, xacro)
@@ -118,6 +118,43 @@
     </joint>
     <link name="${name}_color_optical_frame"/>
+    <!-- IMU -->
+    <!-- see datasheet Revision 009, page 114 -->
+    <xacro:property name="d435_imu_px" value="-0.01602"/>
+    <xacro:property name="d435_imu_py" value="-0.03022"/>
+    <xacro:property name="d435_imu_pz" value="+0.0074"/>
+    <link name="${name}_accel_frame" />
+    <link name="${name}_accel_optical_frame" />
+    <link name="${name}_gyro_frame" />
+    <link name="${name}_gyro_optical_frame" />
+    <link name="${name}_imu_optical_frame" />
+    <joint name="${name}_accel_joint" type="fixed">
+      <origin xyz = "${d435_imu_px} ${d435_imu_py} ${d435_imu_pz}" rpy = "0 0 0" />
+      <parent link="${name}_link" />
+      <child link="${name}_accel_frame" />
+    </joint>
+    <joint name="${name}_accel_optical_joint" type="fixed">
+      <origin xyz = "0 0 0" rpy = "${-M_PI/2} 0 ${-M_PI/2}" />
+      <parent link="${name}_accel_frame" />
+      <child link="${name}_accel_optical_frame" />
+    </joint>
+    <joint name="${name}_gyro_joint" type="fixed">
+      <origin xyz = "${d435_imu_px} ${d435_imu_py} ${d435_imu_pz}" rpy = "0 0 0" />
+      <parent link="${name}_link" />
+      <child link="${name}_gyro_frame" />
+    </joint>
+    <joint name="${name}_gyro_optical_joint" type="fixed">
+      <origin xyz = "0 0 0" rpy = "${-M_PI/2} 0 ${-M_PI/2}" />
+      <parent link="${name}_gyro_frame" />
+      <child link="${name}_gyro_optical_frame" />
+    </joint>
+    <joint name="${name}_imu_optical_joint" type="fixed">
+      <origin xyz = "0 0 0" rpy = "0 0 0" />
+      <parent link="${name}_gyro_optical_frame" />
+      <child link="${name}_imu_optical_frame" />
+    </joint>
     <!-- Realsense Gazebo Plugin -->
-    <xacro:gazebo_d435 camera_name="${name}" reference_link="${name}_link" topics_ns="${topics_ns}" depth_optical_frame="${name}_depth_optical_frame" color_optical_frame="${name}_color_optical_frame" infrared1_optical_frame="${name}_left_ir_optical_frame" infrared2_optical_frame="${name}_right_ir_optical_frame" publish_pointcloud="${publish_pointcloud}"/>
+    <xacro:gazebo_d435 camera_name="${name}" reference_link="${name}_link" topics_ns="${topics_ns}" depth_optical_frame="${name}_depth_optical_frame" color_optical_frame="${name}_color_optical_frame" infrared1_optical_frame="${name}_left_ir_optical_frame" infrared2_optical_frame="
+    ${name}_imu_optical_frame" imu_optical_frame="
+    ${name}_right_ir_optical_frame" publish_pointcloud="${publish_pointcloud}"/>
   </xacro:macro>
 </robot>
